File: Palplant.sch (EAGLE design)
At the start: 28 parts, among them IC2 MCP73831/OT, U2 ESP-12E/F

Commit message: The resistor now use the same reference and package
Parts:
- C5, C6: device adafruit:C-USC0805 -> rcl:C-USC0603
- R1, R3, R4, R5, R7, R9: device resistor:R-US_R0805W -> rcl:R-US_R0603
- R14, R15, R16, R20, R6: device Discrete:R-0603 -> rcl:R-US_R0603
Changed lines of the file:
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@@
 <part name="GND9" library="supply1" deviceset="GND" device=""/>
 <part name="P+2" library="supply1" deviceset="VCC" device=""/>
-<part name="R1" library="resistor" deviceset="R-US_" device="R0805W" value="4.7k">
+<part name="R1" library="rcl" deviceset="R-US_" device="R0603" value="4.7k">
 <attribute name="MF" value=""/>
 <attribute name="MPN" value="MC0805S8F4701T5E"/>
 <attribute name="OC_NEWARK" value="79M6093"/>
 </part>
-<part name="R5" library="resistor" deviceset="R-US_" device="R0805W" value="100">
+<part name="R5" library="rcl" deviceset="R-US_" device="R0603" value="100">
 <attribute name="MF" value=""/>
 <attribute name="MPN" value="ERJ-6ENF1002V"/>
@@
 <part name="P+3" library="supply1" deviceset="VCC" device=""/>
 <part name="GND1" library="supply1" deviceset="GND" device=""/>
-<part name="R9" library="resistor" deviceset="R-US_" device="R0805W" value="4.7k">
+<part name="R9" library="rcl" deviceset="R-US_" device="R0603" value="4.7k">
 <attribute name="MF" value=""/>
 <attribute name="MPN" value="MC0805S8F4701T5E"/>
@@
 </part>
 <part name="GND2" library="supply1" deviceset="GND" device=""/>
-<part name="C5" library="adafruit" deviceset="C-US" device="C0805" value="0.1uF">
+<part name="C5" library="rcl" deviceset="C-US" device="C0603" value="0.1uF">
 <attribute name="MF" value=""/>
 <attribute name="MPN" value="0805B104M500CT"/>
@@
 <part name="GND7" library="supply1" deviceset="GND" device=""/>
 <part name="P+7" library="supply1" deviceset="VCC" device=""/>
-<part name="R7" library="resistor" deviceset="R-US_" device="R0805W" value="4.7k">
+<part name="R7" library="rcl" deviceset="R-US_" device="R0603" value="4.7k">
 <attribute name="MF" value=""/>
 <attribute name="MPN" value="MC0805S8F4701T5E"/>
 <attribute name="OC_NEWARK" value="79M6093"/>
 </part>
-<part name="C6" library="adafruit" deviceset="C-US" device="C0805" value="0.1uF">
+<part name="C6" library="rcl" deviceset="C-US" device="C0603" value="0.1uF">
 <attribute name="MF" value=""/>
 <attribute name="MPN" value="0805B104M500CT"/>
@@
 <part name="GND23" library="supply1" deviceset="GND" device=""/>
 <part name="U2" library="Discrete" deviceset="ESP-12E/F" device=""/>
-<part name="R3" library="resistor" deviceset="R-US_" device="R0805W" value="4.7k">
+<part name="R3" library="rcl" deviceset="R-US_" device="R0603" value="4.7k">
 <attribute name="MF" value=""/>
 <attribute name="MPN" value="MC0805S8F4701T5E"/>
@@
 </part>
 <part name="CHG" library="Discrete" deviceset="007-LED*" device="0603" value="ORANGE"/>
-<part name="R6" library="Discrete" deviceset="R*" device="-0603" value="1k"/>
+<part name="R6" library="rcl" deviceset="R-US_" device="R0603" value="1k"/>
 <part name="C8" library="Discrete" deviceset="C*" device="-0603" value="10u"/>
 <part name="IC2" library="adafruit" deviceset="MCP73831" device="/OT"/>
-<part name="R20" library="Discrete" deviceset="R*" device="-0603" value="5k"/>
+<part name="R20" library="rcl" deviceset="R-US_" device="R0603" value="5k"/>
 <part name="J5" library="SparkFun" deviceset="M02" device="-JST-2MM-SMT"/>
 <part name="LDO" library="MCP1700" deviceset="MCP1700T-3302E/TT" device=""/>
@@
 <part name="GND5" library="supply1" deviceset="GND" device=""/>
 <part name="GND10" library="supply1" deviceset="GND" device=""/>
-<part name="R14" library="Discrete" deviceset="R*" device="-0603" value="1K"/>
+<part name="R14" library="rcl" deviceset="R-US_" device="R0603" value="1K"/>
 <part name="L" library="Discrete" deviceset="LED*" device="'0603'" value="BLUE"/>
 <part name="J1" library="SparkFun" deviceset="M02" device="-JST-2MM-SMT"/>
 <part name="J2" library="Connector" deviceset="HEADER-12P" device="-2.54"/>
 <part name="J6" library="Connector" deviceset="HEADER-12P" device="-2.54"/>
-<part name="R4" library="resistor" deviceset="R-US_" device="R0805W" value="4.7k">
+<part name="R4" library="rcl" deviceset="R-US_" device="R0603" value="4.7k">
 <attribute name="MF" value=""/>
 <attribute name="MPN" value="MC0805S8F4701T5E"/>
@@
 </part>
 <part name="GND4" library="supply1" deviceset="GND" device=""/>
-<part name="R15" library="Discrete" deviceset="R*" device="-0603" value="220k/1%"/>
-<part name="R16" library="Discrete" deviceset="R*" device="-0603" value="100K/1%"/>
+<part name="R15" library="rcl" deviceset="R-US_" device="R0603" value="220k/1%"/>
+<part name="R16" library="rcl" deviceset="R-US_" device="R0603" value="100K/1%"/>
 </parts>
 <sheets>
@@
 <attribute name="VALUE" x="69.85" y="63.5" size="1.016" layer="96" rot="R270"/>
 </instance>
-<instance part="R6" gate="R" x="82.55" y="57.15" smashed="yes">
+<instance part="R6" gate="G$1" x="82.55" y="57.15" smashed="yes">
 <attribute name="NAME" x="78.74" y="58.42" size="1.016" layer="95" ratio="10"/>
 <attribute name="VALUE" x="82.55" y="58.42" size="1.016" layer="96" ratio="10"/>
@@
 <instance part="C8" gate="C" x="64.77" y="59.69" rot="R90"/>
 <instance part="IC2" gate="G$1" x="102.87" y="62.23"/>
-<instance part="R20" gate="R" x="130.81" y="62.23" smashed="yes">
+<instance part="R20" gate="G$1" x="130.81" y="62.23" smashed="yes">
 <attribute name="NAME" x="127" y="62.23" size="1.016" layer="95" ratio="10"/>
 <attribute name="VALUE" x="130.81" y="64.77" size="1.016" layer="96" ratio="10" rot="R180"/>
@@
 <instance part="GND5" gate="1" x="64.77" y="46.99"/>
 <instance part="GND10" gate="1" x="118.11" y="73.66" rot="R270"/>
-<instance part="R14" gate="R" x="121.92" y="15.24" rot="R180"/>
+<instance part="R14" gate="G$1" x="121.92" y="15.24" rot="R180"/>
 <instance part="L" gate="LED" x="133.35" y="15.24"/>
 <instance part="J1" gate="G$1" x="33.02" y="68.58" smashed="yes" rot="R180">
@@
 </instance>
 <instance part="GND4" gate="1" x="162.56" y="111.76" rot="R90"/>
-<instance part="R15" gate="R" x="125.73" y="93.98" rot="R180"/>
-<instance part="R16" gate="R" x="147.32" y="93.98" rot="R180"/>
+<instance part="R15" gate="G$1" x="125.73" y="93.98" rot="R180"/>
+<instance part="R16" gate="G$1" x="147.32" y="93.98" rot="R180"/>
 </instances>
 <busses>
@@
 </segment>
 <segment>
-<pinref part="R20" gate="R" pin="2"/>
-<wire x1="134.62" y1="62.23" x2="139.7" y2="62.23" width="0.1524" layer="91"/>
+<pinref part="R20" gate="G$1" pin="2"/>
+<wire x1="135.89" y1="62.23" x2="139.7" y2="62.23" width="0.1524" layer="91"/>
 <wire x1="139.7" y1="62.23" x2="139.7" y2="57.15" width="0.1524" layer="91"/>
 <pinref part="IC2" gate="G$1" pin="VSS"/>
@@
 </segment>
 <segment>
-<pinref part="R16" gate="R" pin="1"/>
-<wire x1="151.13" y1="93.98" x2="162.56" y2="93.98" width="0.1524" layer="91"/>
+<pinref part="R16" gate="G$1" pin="1"/>
+<wire x1="152.4" y1="93.98" x2="162.56" y2="93.98" width="0.1524" layer="91"/>
 <label x="163.83" y="93.98" size="1.778" layer="95" rot="R180"/>
 </segment>
@@
 <segment>
 <pinref part="CHG" gate="LED" pin="-"/>
-<pinref part="R6" gate="R" pin="1"/>
-<wire x1="73.66" y1="57.15" x2="78.74" y2="57.15" width="0.1524" layer="91"/>
+<pinref part="R6" gate="G$1" pin="1"/>
+<wire x1="73.66" y1="57.15" x2="77.47" y2="57.15" width="0.1524" layer="91"/>
 </segment>
 </net>
 <net name="N$20" class="0">
 <segment>
-<pinref part="R6" gate="R" pin="2"/>
+<pinref part="R6" gate="G$1" pin="2"/>
 <pinref part="IC2" gate="G$1" pin="STAT"/>
-<wire x1="86.36" y1="57.15" x2="90.17" y2="57.15" width="0.1524" layer="91"/>
+<wire x1="87.63" y1="57.15" x2="90.17" y2="57.15" width="0.1524" layer="91"/>
 </segment>
 </net>
@@
 <segment>
 <pinref part="IC2" gate="G$1" pin="PROG"/>
-<pinref part="R20" gate="R" pin="1"/>
-<wire x1="118.11" y1="62.23" x2="127" y2="62.23" width="0.1524" layer="91"/>
+<pinref part="R20" gate="G$1" pin="1"/>
+<wire x1="118.11" y1="62.23" x2="125.73" y2="62.23" width="0.1524" layer="91"/>
 </segment>
 </net>
@@
 <segment>
 <pinref part="L" gate="LED" pin="+"/>
-<pinref part="R14" gate="R" pin="1"/>
-<wire x1="125.73" y1="15.24" x2="129.54" y2="15.24" width="0.1524" layer="91"/>
+<pinref part="R14" gate="G$1" pin="1"/>
+<wire x1="127" y1="15.24" x2="129.54" y2="15.24" width="0.1524" layer="91"/>
 </segment>
 </net>
@@
 </segment>
 <segment>
-<pinref part="R14" gate="R" pin="2"/>
+<pinref part="R14" gate="G$1" pin="2"/>
 <label x="107.95" y="12.7" size="1.4224" layer="95" ratio="10"/>
-<wire x1="118.11" y1="15.24" x2="109.22" y2="15.24" width="0.1524" layer="91"/>
+<wire x1="116.84" y1="15.24" x2="109.22" y2="15.24" width="0.1524" layer="91"/>
 </segment>
 </net>
@@
 </segment>
 <segment>
-<pinref part="R15" gate="R" pin="1"/>
-<pinref part="R16" gate="R" pin="2"/>
-<wire x1="129.54" y1="93.98" x2="133.35" y2="93.98" width="0.1524" layer="91"/>
-<wire x1="133.35" y1="93.98" x2="143.51" y2="93.98" width="0.1524" layer="91"/>
+<pinref part="R15" gate="G$1" pin="1"/>
+<pinref part="R16" gate="G$1" pin="2"/>
+<wire x1="130.81" y1="93.98" x2="133.35" y2="93.98" width="0.1524" layer="91"/>
+<wire x1="133.35" y1="93.98" x2="142.24" y2="93.98" width="0.1524" layer="91"/>
 <wire x1="133.35" y1="93.98" x2="133.35" y2="102.87" width="0.1524" layer="91"/>
 <label x="133.35" y="97.79" size="1.778" layer="95" rot="R90"/>
@@
 </segment>
 <segment>
-<pinref part="R15" gate="R" pin="2"/>
-<wire x1="121.92" y1="93.98" x2="110.49" y2="93.98" width="0.1524" layer="91"/>
+<pinref part="R15" gate="G$1" pin="2"/>
+<wire x1="120.65" y1="93.98" x2="110.49" y2="93.98" width="0.1524" layer="91"/>
 <label x="119.38" y="96.52" size="1.778" layer="95" rot="R180"/>
 </segment>
